File: LM2670-ADJ-Carrier-Set-SMD/LM2670-ADJ-Carrier-Set-SMD.kicad_pcb (KiCad board)
At the start: 2 copper layers, 19.6 x 32.4 mm, 11 parts, among them IC1 LM2670SX-3.3_NOPB, J1 Conn_01x03

Commit message: ADJ Carrier SMD
Parts:
- C3, C4: footprint Capacitor_SMD:C_0603_1608Metric_Pad1.08x0.95mm_HandSolder -> Capacitor_SMD:C_1206_3216Metric_Pad1.33x1.80mm_HandSolder
- R2, R3: footprint Resistor_SMD:R_0612_1632Metric_Pad1.18x3.40mm_HandSolder -> Resistor_SMD:R_1206_3216Metric_Pad1.30x1.75mm_HandSolder
- moved C4 3.07 mm to (139.0, 103.7)
- moved D1 2.47 mm to (143.9, 103.5)
- moved R2 0.52 mm to (144.7, 90.0)
Routing:
- net GND: track 44.1 -> 38.4 mm, vias 2 -> 3
- net Net-(J1-Pin_2): track 59.6 -> 64.2 mm
- net +VDC: track 60.8 -> 57.2 mm
- net Net-(IC1-FEEDBACK/FB): track 12.7 -> 11.9 mm
- net Net-(IC1-SWITCH_OUTPUT): track 37.1 -> 37.4 mm, vias 1 -> 2
Other:
- board text added: "GND"
- board text added: "VDC"
- board text added: "VO"
