File: LM2670-ADJ-Carrier/LM2670-ADJ-Carrier.kicad_pcb (KiCad board)
At the start: 2 copper layers, 19.6 x 32.4 mm, 11 parts, among them IC1 LM2670SX-3.3_NOPB, J1 Conn_01x03

Commit message: finished ADJ board and adding the Fab Files for it.
Parts:
- moved R2 6.64 mm to (144.2, 90.0)
- moved R3 6.64 mm to (139.7, 90.0)
- moved D1 2.88 mm to (141.5, 104.1)
- moved C4 2.08 mm to (136.6, 101.8)
- moved C3 1.89 mm to (139.6, 95.0)
Routing:
- net Net-(J1-Pin_2): track 12.8 -> 54.7 mm
- net +VDC: track 20.9 -> 60.8 mm
- net Net-(IC1-SWITCH_OUTPUT): track 2.73 -> 29.5 mm
- net GND: track 35.1 -> 47.8 mm, vias 1 -> 2
- net Net-(IC1-FEEDBACK/FB): track 2.83 -> 12.7 mm, vias 0 -> 1
- net Net-(IC1-CBOOST/CB): track 3.25 -> 4.55 mm
Other:
- board text added: "LM2670SX Adjustable"
- board text removed: "LM2670SX"

Commit message: update footprints in schematic only
Parts:
- C3, C4: footprint Capacitor_SMD:C_0603_1608Metric_Pad1.08x0.95mm_HandSolder -> Capacitor_SMD:C_1206_3216Metric_Pad1.33x1.80mm_HandSolder
- R2, R3: footprint Resistor_SMD:R_0612_1632Metric_Pad1.18x3.40mm_HandSolder -> Resistor_SMD:R_1206_3216Metric_Pad1.30x1.75mm_HandSolder
- moved C4 2.06 mm to (138.0, 103.3)
- moved D1 1.22 mm to (142.5, 104.9)
Routing:
- net +VDC: track 60.8 -> 58.9 mm
- net GND: track 47.8 -> 46.5 mm
- net Net-(IC1-FEEDBACK/FB): track 12.7 -> 11.6 mm
Other:
- board text added: "GND"
- board text added: "VDC"
- board text added: "VO"

Commit message: Update to ADJ-Carrier - PCB and Fab Files - Added ibom.html
Parts:
- moved R2 0.56 mm to (144.8, 89.9)
Changed lines of the file:
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@@
 	(footprint "Resistor_SMD:R_1206_3216Metric_Pad1.30x1.75mm_HandSolder"
 		(layer "B.Cu")
-		(at 144.224819 89.98109 180)
+		(at 144.782452 89.949036 180)
 		(descr "Resistor SMD 1206 (3216 Metric), square (rectangular) end terminal, IPC_7351 nominal with elongated pad for handsoldering. (Body size source: IPC-SM-782 page 72, https://www.pcb-3d.com/wordpress/wp-content/uploads/ipc-sm-782a_amendment_1_and_2.pdf), generated with kicad-footprint-generator")
 		(tags "resistor handsolder")
@@
 	(footprint "Resistor_SMD:R_1206_3216Metric_Pad1.30x1.75mm_HandSolder"
 		(layer "B.Cu")
-		(at 139.716067 89.98109 180)
+		(at 139.731542 89.960489 180)
 		(descr "Resistor SMD 1206 (3216 Metric), square (rectangular) end terminal, IPC_7351 nominal with elongated pad for handsoldering. (Body size source: IPC-SM-782 page 72, https://www.pcb-3d.com/wordpress/wp-content/uploads/ipc-sm-782a_amendment_1_and_2.pdf), generated with kicad-footprint-generator")
 		(tags "resistor handsolder")
@@
 	)
 	(segment
-		(start 145.774819 89.98109)
-		(end 143.217459 89.98109)
+		(start 146.332452 89.949036)
+		(end 143.249513 89.949036)
+		(width 0.762)
+		(layer "F.Cu")
+		(net 2)
+	)
+	(segment
+		(start 143.249513 89.949036)
+		(end 142.161749 91.0368)
 		(width 0.762)
 		(layer "F.Cu")
@@
 	)
 	(segment
-		(start 143.217459 89.98109)
-		(end 142.161749 91.0368)
-		(width 0.762)
-		(layer "F.Cu")
-		(net 2)
-	)
-	(segment
 		(start 140.312678 104.899059)
 		(end 140.465476 104.899059)
@@
 	)
 	(via
-		(at 145.774819 89.98109)
+		(at 146.332452 89.949036)
 		(size 0.8)
 		(drill 0.4)
@@
 	)
 	(segment
-		(start 145.903425 89.852484)
-		(end 145.774819 89.98109)
-		(width 0.762)
-		(layer "B.Cu")
-		(net 2)
-	)
-	(segment
 		(start 150.650694 89.852484)
 		(end 150.650694 94.078245)
@@
 		(start 150.522088 89.98109)
 		(end 150.650694 89.852484)
+		(width 0.762)
+		(layer "B.Cu")
+		(net 2)
+	)
+	(segment
+		(start 146.332452 89.949036)
+		(end 146.429004 89.852484)
 		(width 0.762)
 		(layer "B.Cu")
@@
 	)
 	(segment
-		(start 150.650694 89.852484)
-		(end 145.903425 89.852484)
+		(start 146.429004 89.852484)
+		(end 150.650694 89.852484)
 		(width 0.762)
 		(layer "B.Cu")
@@
 	)
 	(segment
+		(start 138.402294 89.960489)
+		(end 138.181542 89.960489)
+		(width 0.762)
+		(layer "B.Cu")
+		(net 5)
+	)
+	(segment
 		(start 151.678449 101.550349)
 		(end 145.30817 101.550349)
@@
 	)
 	(segment
-		(start 143.468452 95.026647)
-		(end 138.422895 89.98109)
-		(width 0.762)
-		(layer "B.Cu")
-		(net 5)
-	)
-	(segment
 		(start 143.468452 99.710631)
 		(end 143.468452 95.026647)
@@
 	)
 	(segment
+		(start 143.468452 95.026647)
+		(end 138.402294 89.960489)
+		(width 0.762)
+		(layer "B.Cu")
+		(net 5)
+	)
+	(segment
 		(start 151.678449 113.299142)
 		(end 152.811683 114.432376)
@@
 		(start 151.678449 100.508)
 		(end 151.678449 101.550349)
-		(width 0.762)
-		(layer "B.Cu")
-		(net 5)
-	)
-	(segment
-		(start 138.422895 89.98109)
-		(end 138.166067 89.98109)
 		(width 0.762)
 		(layer "B.Cu")
@@
 	)
 	(segment
-		(start 142.674819 89.98109)
-		(end 141.266067 89.98109)
+		(start 143.232452 89.949036)
+		(end 141.292995 89.949036)
 		(width 0.762)
 		(layer "B.Cu")
@@
 	)
 	(segment
-		(start 142.674819 91.527299)
-		(end 142.674819 89.98109)
+		(start 144.645369 93.497849)
+		(end 143.232452 92.084932)
+		(width 0.762)
+		(layer "B.Cu")
+		(net 7)
+	)
+	(segment
+		(start 143.232452 92.084932)
+		(end 143.232452 89.949036)
 		(width 0.762)
 		(layer "B.Cu")
@@
 	)
 	(segment
-		(start 144.645369 93.497849)
-		(end 142.674819 91.527299)
-		(width 0.762)
-		(layer "B.Cu")
+		(start 141.292995 89.949036)
+		(end 141.281542 89.960489)
+		(width 0.762)
+		(layer "B.Cu")
