File: LM2670SX-Carrier/LM2670SX-Carrier.kicad_pcb (KiCad board)
At the start: 2 copper layers, 19.6 x 32.4 mm, 10 parts, among them IC1 LM2670SX-3.3_NOPB, J1 Conn_01x03

Commit message: rename
Other:
- board text added: "LM2670SX"
- board text removed: "3.3V 1.0A LM2670SX"
Changed lines of the file:
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@@
   (gr_line (start 170.942 116.84) (end 170.942 84.455)
     (stroke (width 0.1) (type solid)) (layer "Edge.Cuts"))
-  (gr_text "3.3V 1.0A\nLM2670SX" (at 190.126311 112.574941 90) (layer "F.SilkS")
+  (gr_text "LM2670SX" (at 190.126311 112.574941 90) (layer "F.SilkS")
     (effects (font (size 1 1) (thickness 0.15)) (justify left bottom))
   )

Commit message: update reg carrier
Parts:
- C3, C4: footprint Capacitor_SMD:C_0603_1608Metric_Pad1.08x0.95mm_HandSolder -> Capacitor_SMD:C_1206_3216Metric_Pad1.33x1.80mm_HandSolder
- R1: footprint Resistor_SMD:R_0612_1632Metric_Pad1.18x3.40mm_HandSolder -> Resistor_SMD:R_1206_3216Metric_Pad1.30x1.75mm_HandSolder
- moved C4 4.08 mm to (173.7, 103.3)
- moved C3 3.25 mm to (174.8, 93.3)
- moved D2 3.09 mm to (179.0, 103.3)
- moved R1 2.84 mm to (180.6, 93.4)
Routing:
- net +VDC: track 37.4 -> 43.3 mm
- net Net-(IC1-SWITCH_OUTPUT): track 22.1 -> 27.8 mm
- net Net-(IC1-SYNC): track 3.90 -> 7.09 mm
- net Net-(IC1-CBOOST/CB): track 3.07 -> 5.94 mm
Other:
- board text added: "GND"
- board text added: "VDC"
- board text added: "VO"
